Commit message: [update]07

File: urdf/06-flexible.urdf (robot description, URDF)
Before this commit: robot visual, 16 links, 15 joints
Joints:
- joint gripper_extension: limit (none) -> lower=-0.38 upper=0 effort=1000.0 velocity=0.5; type fixed -> prismatic
- joint left_front_wheel_joint: axis (none) -> 0 1 0; type fixed -> continuous
- joint left_gripper_joint: axis (none) -> 0 0 1; limit (none) -> lower=0 upper=0.548 effort=1000.0 velocity=0.5; type fixed -> revolute
- joint right_gripper_joint: axis (none) -> 0 0 -1; limit (none) -> lower=0.0 upper=0.548 effort=1000.0 velocity=0.5
