Commit message: [add&update] it is possible to launch gazebo with R2D2

File: urdf/09-publishjoints.urdf.xacro (robot description, xacro)
@@ -1,4 +1,4 @@
 <?xml version="1.0"?>
-<robot name="macroed" xmlns:xacro="http://ros.org/wiki/xacro">
+<robot name="gazebo_robot" xmlns:xacro="http://ros.org/wiki/xacro">
 	<xacro:property name="width" value="0.2" />
 	<xacro:property name="leglen" value="0.6"/>
@@ -18,8 +18,8 @@
 	</material>
 	<xacro:macro name="default_inertial" params="mass">
-		<inertia>
+		<inertial>
 			<mass value="${mass}" />
 			<inertia ixx="1.0" ixy="0.0" ixz="0.0" iyy="1.0" iyz="0.0" izz="1.0" />
-		</inertia>
+		</inertial>
 	</xacro:macro>
 	<link name="base_link">
@@ -214,3 +214,10 @@
 		<origin xyz="${.707*width+0.04} 0 ${.707*width}"/>
 	</joint>
+	<!--Gazebo plugin for ROS Control -->
+	<!--Joint state publisher in Gazebo-->
+	<gazebo>
+		<plugin name="gazebo_ros_control" filename="libgazebo_ros_control.so">
+			<robotNameSpace>/</robotNameSpace>
+		</plugin>
+	</gazebo>
 </robot>

Commit message: [update]

File: urdf/09-publishjoints.urdf.xacro (robot description, xacro)
@@ -216,4 +216,5 @@
 	<!--Gazebo plugin for ROS Control -->
 	<!--Joint state publisher in Gazebo-->
+	<!--Connection between ROS and gazebo-->
 	<gazebo>
 		<plugin name="gazebo_ros_control" filename="libgazebo_ros_control.so">

File: urdf/model.urdf (robot description, URDF)
Before this commit: robot macroed, 16 links, 15 joints
Links:
- link base_link: mass None -> 10
- link box: mass None -> 1
- link gripper_pole: mass None -> 0.05
- link head: mass None -> 2
- link left_back_wheel: mass None -> 1.0
- link left_base: mass None -> 10
- link left_front_wheel: mass None -> 1.0
- link left_gripper: mass None -> 0.05
- link left_leg: mass None -> 10
- link left_tip: mass None -> 0.05
- link right_back_wheel: mass None -> 1.0
- link right_base: mass None -> 10
- link right_front_wheel: mass None -> 1.0
- link right_gripper: mass None -> 0.05
- link right_leg: mass None -> 10
- link right_tip: mass None -> 0.05
